File: prints/sensor/sensorshield/sensorshield/sensorshield.kicad_pcb (KiCad board)
At the start: 2 copper layers, 30.5 x 17 mm, 6 parts, among them J2 RaspberryHall

Commit message: updated schematics and prints
Parts:
- added R3: 6k8, Resistor_SMD:R_0805_2012Metric_Pad1.20x1.40mm_HandSolder, F.Cu at (135.5, 115.0)
- added R4: 10, Resistor_SMD:R_0805_2012Metric_Pad1.20x1.40mm_HandSolder, F.Cu at (135.5, 117.0)
- moved R1 8.51 mm to (139.5, 117.0)
- moved R2 8.51 mm to (139.5, 115.0)
- moved G*** 7.02 mm to (137.0, 124.0)
- moved J2 0.50 mm to (147.0, 125.8)
Connections:
- U1 pad 3: +5V -> Net-(U1-ADR)
- U1 pad 4: GND -> +5V
Routing:
- net Net-(U1-ADR): track 0.00 -> 15.2 mm
- net GND: track 0.00 -> 11.5 mm, vias 0 -> 5
- net Net-(J2-Pin_3): track 50.3 -> 42.8 mm
- net +5V: track 30.2 -> 26.5 mm
Other:
- board text added: "ADR"
