File: prints/sensor/sensorshield/sensorshield/sensorshield.kicad_sch (KiCad schematic)
At the start: 5 parts, among them J2 RaspberryHall

Commit message: updated schematics and prints
Parts:
- added R3: 6k8, Resistor_SMD:R_0805_2012Metric_Pad1.20x1.40mm_HandSolder, symbol Device:R
- added R4: 0, Resistor_SMD:R_0805_2012Metric_Pad1.20x1.40mm_HandSolder, symbol Device:R
Connections:
- net +5V: now also U1.4 (VDD), R4.1; no longer U1.3 (ADR)
- net GND: now also R3.2; no longer U1.4 (VDD)
- new net: R3.1, R4.2, U1.3 (ADR)
Changed lines of the file:
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@@
   (junction (at 113.03 40.005) (diameter 0) (color 0 0 0 0)
   )
+  (junction (at 78.74 43.815) (diameter 0) (color 0 0 0 0)
+  )
+  (wire (pts (xy 117.475 21.59) (xy 117.475 22.86))
+    (stroke (width 0) (type default))
+  )
   (wire (pts (xy 121.92 38.1) (xy 121.92 43.815))
     (stroke (width 0) (type default))
   )
+  (wire (pts (xy 78.74 21.59) (xy 78.74 31.115))
+    (stroke (width 0) (type default))
+  )
   (wire (pts (xy 113.03 38.1) (xy 113.03 40.005))
     (stroke (width 0) (type default))
   )
+  (wire (pts (xy 65.405 47.625) (xy 85.725 47.625))
+    (stroke (width 0) (type default))
+  )
+  (wire (pts (xy 78.74 55.88) (xy 78.74 43.815))
+    (stroke (width 0) (type default))
+  )
   (wire (pts (xy 121.92 22.86) (xy 121.92 30.48))
     (stroke (width 0) (type default))
@@
     (stroke (width 0) (type default))
   )
-  (wire (pts (xy 65.405 47.625) (xy 81.915 47.625))
-    (stroke (width 0) (type default))
-  )
-  (wire (pts (xy 65.405 40.005) (xy 65.405 47.625))
-    (stroke (width 0) (type default))
-  )
-  (wire (pts (xy 81.915 43.815) (xy 81.915 47.625))
+  (wire (pts (xy 65.405 21.59) (xy 65.405 47.625))
+    (stroke (width 0) (type default))
+  )
+  (wire (pts (xy 65.405 47.625) (xy 65.405 55.245))
     (stroke (width 0) (type default))
   )
@@
     (stroke (width 0) (type default))
   )
-  (wire (pts (xy 65.405 47.625) (xy 65.405 55.245))
+  (wire (pts (xy 78.74 43.815) (xy 85.725 43.815))
+    (stroke (width 0) (type default))
+  )
+  (wire (pts (xy 78.74 38.735) (xy 78.74 43.815))
     (stroke (width 0) (type default))
   )
@@
   )
   (wire (pts (xy 117.475 22.86) (xy 113.03 22.86))
-    (stroke (width 0) (type default))
-  )
-  (wire (pts (xy 85.725 43.815) (xy 81.915 43.815))
     (stroke (width 0) (type default))
   )
@@
     )
   )
-  (symbol (lib_id "power:+5V") (at 65.405 40.005 0) (unit 1)
-    (in_bom yes) (on_board yes) (dnp no) (fields_autoplaced)
-    (property "Reference" "#PWR02" (at 65.405 43.815 0)
-      (effects (font (size 1.27 1.27)) hide)
-    )
-    (property "Value" "+5V" (at 65.405 35.56 0)
-      (effects (font (size 1.27 1.27)))
-    )
-    (property "Footprint" "" (at 65.405 40.005 0)
-      (effects (font (size 1.27 1.27)) hide)
-    )
-    (property "Datasheet" "" (at 65.405 40.005 0)
+  (symbol (lib_id "power:+5V") (at 65.405 21.59 0) (unit 1)
+    (in_bom yes) (on_board yes) (dnp no) (fields_autoplaced)
+    (property "Reference" "#PWR02" (at 65.405 25.4 0)
+      (effects (font (size 1.27 1.27)) hide)
+    )
+    (property "Value" "+5V" (at 65.405 17.145 0)
+      (effects (font (size 1.27 1.27)))
+    )
+    (property "Footprint" "" (at 65.405 21.59 0)
+      (effects (font (size 1.27 1.27)) hide)
+    )
+    (property "Datasheet" "" (at 65.405 21.59 0)
       (effects (font (size 1.27 1.27)) hide)
     )
@@
     )
   )
+  (symbol (lib_id "Device:R") (at 78.74 59.69 0) (unit 1)
+    (in_bom yes) (on_board yes) (dnp no) (fields_autoplaced)
+    (property "Reference" "R3" (at 81.28 58.42 0)
+      (effects (font (size 1.27 1.27)) (justify left))
+    )
+    (property "Value" "6k8" (at 81.28 60.96 0)
+      (effects (font (size 1.27 1.27)) (justify left))
+    )
+    (property "Footprint" "Resistor_SMD:R_0805_2012Metric_Pad1.20x1.40mm_HandSolder" (at 76.962 59.69 90)
+      (effects (font (size 1.27 1.27)) hide)
+    )
+    (property "Datasheet" "~" (at 78.74 59.69 0)
+      (effects (font (size 1.27 1.27)) hide)
+    )
+    (pin "2")
+    (pin "1")
+    (instances
+      (project "sensorshield"
+        (path "/dbe6534e-7a5a-40d6-a240-b2690612024e"
+          (reference "R3") (unit 1)
+        )
+      )
+    )
+  )
+  (symbol (lib_id "Device:R") (at 78.74 34.925 0) (unit 1)
+    (in_bom yes) (on_board yes) (dnp no) (fields_autoplaced)
+    (property "Reference" "R4" (at 81.28 33.655 0)
+      (effects (font (size 1.27 1.27)) (justify left))
+    )
+    (property "Value" "0" (at 81.28 36.195 0)
+      (effects (font (size 1.27 1.27)) (justify left))
+    )
+    (property "Footprint" "Resistor_SMD:R_0805_2012Metric_Pad1.20x1.40mm_HandSolder" (at 76.962 34.925 90)
+      (effects (font (size 1.27 1.27)) hide)
+    )
+    (property "Datasheet" "~" (at 78.74 34.925 0)
+      (effects (font (size 1.27 1.27)) hide)
+    )
+    (pin "2")
+    (pin "1")
+    (instances
+      (project "sensorshield"
+        (path "/dbe6534e-7a5a-40d6-a240-b2690612024e"
+          (reference "R4") (unit 1)
+        )
+      )
+    )
+  )
   (symbol (lib_id "Device:C") (at 65.405 59.055 0) (unit 1)
-    (in_bom yes) (on_board yes) (dnp no) (fields_autoplaced)
+    (in_bom yes) (on_board yes) (dnp no)
     (property "Reference" "C1" (at 68.58 57.785 0)
       (effects (font (size 1.27 1.27)) (justify left))
     )
-    (property "Value" "100nF" (at 68.58 60.325 0)
+    (property "Value" "100nF" (at 68.58 59.69 0)
       (effects (font (size 1.27 1.27)) (justify left))
     )
@@
     )
   )
-  (symbol (lib_id "power:GND") (at 85.725 47.625 0) (unit 1)
-    (in_bom yes) (on_board yes) (dnp no) (fields_autoplaced)
-    (property "Reference" "#PWR010" (at 85.725 53.975 0)
-      (effects (font (size 1.27 1.27)) hide)
-    )
-    (property "Value" "GND" (at 85.725 52.07 0)
-      (effects (font (size 1.27 1.27)))
-    )
-    (property "Footprint" "" (at 85.725 47.625 0)
-      (effects (font (size 1.27 1.27)) hide)
-    )
-    (property "Datasheet" "" (at 85.725 47.625 0)
+  (symbol (lib_id "power:GND") (at 65.405 62.865 0) (unit 1)
+    (in_bom yes) (on_board yes) (dnp no) (fields_autoplaced)
+    (property "Reference" "#PWR01" (at 65.405 69.215 0)
+      (effects (font (size 1.27 1.27)) hide)
+    )
+    (property "Value" "GND" (at 65.405 67.31 0)
+      (effects (font (size 1.27 1.27)))
+    )
+    (property "Footprint" "" (at 65.405 62.865 0)
+      (effects (font (size 1.27 1.27)) hide)
+    )
+    (property "Datasheet" "" (at 65.405 62.865 0)
+      (effects (font (size 1.27 1.27)) hide)
+    )
+    (pin "1")
+    (instances
+      (project "sensorshield"
+        (path "/dbe6534e-7a5a-40d6-a240-b2690612024e"
+          (reference "#PWR01") (unit 1)
+        )
+      )
+    )
+  )
+  (symbol (lib_id "power:GND") (at 78.74 63.5 0) (unit 1)
+    (in_bom yes) (on_board yes) (dnp no) (fields_autoplaced)
+    (property "Reference" "#PWR010" (at 78.74 69.85 0)
+      (effects (font (size 1.27 1.27)) hide)
+    )
+    (property "Value" "GND" (at 78.74 67.945 0)
+      (effects (font (size 1.27 1.27)))
+    )
+    (property "Footprint" "" (at 78.74 63.5 0)
+      (effects (font (size 1.27 1.27)) hide)
+    )
+    (property "Datasheet" "" (at 78.74 63.5 0)
       (effects (font (size 1.27 1.27)) hide)
     )
@@
     )
   )
-  (symbol (lib_id "power:GND") (at 65.405 62.865 0) (unit 1)
-    (in_bom yes) (on_board yes) (dnp no) (fields_autoplaced)
-    (property "Reference" "#PWR01" (at 65.405 69.215 0)
-      (effects (font (size 1.27 1.27)) hide)
-    )
-    (property "Value" "GND" (at 65.405 67.31 0)
-      (effects (font (size 1.27 1.27)))
-    )
-    (property "Footprint" "" (at 65.405 62.865 0)
-      (effects (font (size 1.27 1.27)) hide)
-    )
-    (property "Datasheet" "" (at 65.405 62.865 0)
-      (effects (font (size 1.27 1.27)) hide)
-    )
-    (pin "1")
-    (instances
-      (project "sensorshield"
-        (path "/dbe6534e-7a5a-40d6-a240-b2690612024e"
-          (reference "#PWR01") (unit 1)
+  (symbol (lib_id "power:+5V") (at 78.74 21.59 0) (unit 1)
+    (in_bom yes) (on_board yes) (dnp no) (fields_autoplaced)
+    (property "Reference" "#PWR011" (at 78.74 25.4 0)
+      (effects (font (size 1.27 1.27)) hide)
+    )
+    (property "Value" "+5V" (at 78.74 17.145 0)
+      (effects (font (size 1.27 1.27)))
+    )
+    (property "Footprint" "" (at 78.74 21.59 0)
+      (effects (font (size 1.27 1.27)) hide)
+    )
+    (property "Datasheet" "" (at 78.74 21.59 0)
+      (effects (font (size 1.27 1.27)) hide)
+    )
+    (pin "1")
+    (instances
+      (project "sensorshield"
+        (path "/dbe6534e-7a5a-40d6-a240-b2690612024e"
+          (reference "#PWR011") (unit 1)
         )
       )
@@
     )
   )
-  (symbol (lib_id "power:+5V") (at 117.475 22.86 0) (unit 1)
-    (in_bom yes) (on_board yes) (dnp no) (fields_autoplaced)
-    (property "Reference" "#PWR06" (at 117.475 26.67 0)
-      (effects (font (size 1.27 1.27)) hide)
-    )
-    (property "Value" "+5V" (at 117.475 18.415 0)
-      (effects (font (size 1.27 1.27)))
-    )
-    (property "Footprint" "" (at 117.475 22.86 0)
-      (effects (font (size 1.27 1.27)) hide)
-    )
-    (property "Datasheet" "" (at 117.475 22.86 0)
-      (effects (font (size 1.27 1.27)) hide)
-    )
+  (symbol (lib_id "power:+5V") (at 117.475 21.59 0) (unit 1)
+    (in_bom yes) (on_board yes) (dnp no) (fields_autoplaced)
+    (property "Reference" "#PWR06" (at 117.475 25.4 0)
+      (effects (font (size 1.27 1.27)) hide)
+    )
+    (property "Value" "+5V" (at 117.475 17.145 0)
+      (effects (font (size 1.27 1.27)))
+    )
+    (property "Footprint" "" (at 117.475 21.59 0)
+      (effects (font (size 1.27 1.27)) hide)
+    )
+    (property "Datasheet" "" (at 117.475 21.59 0)
+      (effects (font (size 1.27 1.27)) hide)
+    )
