File: schemata/Hauptschema/mainschematic/hallsensor.kicad_sch (KiCad schematic)
At the start: 0 parts

Commit message: added Revision 0.2.1 of Skógahöf Mainschematic
Parts:
- added C1: 100nF, Capacitor_SMD:C_0805_2012Metric_Pad1.18x1.45mm_HandSolder, symbol Device:C
- added J6: RaspberryHall, TerminalBlock_4Ucon:TerminalBlock_4Ucon_1x04_P3.50mm_Vertical, symbol Connector:Screw_Terminal_01x04
- added R4: 0, Resistor_SMD:R_0805_2012Metric_Pad1.20x1.40mm_HandSolder, symbol Device:R
- added R5, R6, R7: 6k8, Resistor_SMD:R_0805_2012Metric_Pad1.20x1.40mm_HandSolder, symbol Device:R
- added U1: ~, Package_SO:SOIC-8_3.9x4.9mm_P1.27mm, symbol OSRAM_AS5510_DSOM:AS5510-DSOM
Connections:
- new net: R4.2, R5.1, U1.3 (ADR)
- new net +5V: C1.1, J6.1 (Pin_1), R4.1, R6.1, R7.1, U1.4 (VDD)
- new net GND: C1.2, J6.4 (Pin_4), R5.2, U1.1 (NC), U1.2 (VSS), U1.5 (TEST), U1.8 (NC)
- new net SCL: J6.2 (Pin_2), R6.2, U1.7 (SCL)
- new net SDA: J6.3 (Pin_3), R7.2, U1.6 (SDA)
Other:
- note added: "1.0"
- note added: "22.03.24"
- note added: "Hallsensor Module PREN2 Skógahöf"
