File: schemata/Hauptschema/mainschematic/mainschematic.kicad_sch (KiCad schematic)
At the start: 4 parts, among them M1 Stepper_Motor_bipolar, M2 Stepper_Motor_bipolar

Commit message: added Revision 0.2.1 of Skógahöf Mainschematic
Parts:
- added CurrentSensor1: ~, symbol Raspberry_4B:CurrentSensor
Connections:
- net Displayshield/CurrentOut: now also CurrentSensor1.2 (MeasOut)
- net Displayshield/DB4: now also RASPBERRYPI4B1.36 (GPIO_16)
- net Displayshield/DB5: now also RASPBERRYPI4B1.35 (GPIO_19_(PCM_FS))
- net Displayshield/DB6: now also RASPBERRYPI4B1.38 (GPIO_20_(PCM_DIN))
- net Displayshield/DB7: now also RASPBERRYPI4B1.40 (GPIO_21_(PCM_DOUT))
- net Displayshield/E: now also RASPBERRYPI4B1.19 (GPIO_10_(SPI0_MOSI))
- net Displayshield/GND_PASS: now also CurrentSensor1.3 (GND)
- net Displayshield/RS: now also RASPBERRYPI4B1.21 (GPIO_9_(SPI0_MISO))
- net Displayshield/VCC_PASS: now also CurrentSensor1.1 (VDD)
- net +12V: now reaches MotorHAT1.1 (5-12VDC_IN)
- net Earth: now reaches MotorHAT1.2 (GND)
- net +5V: now reaches RASPBERRYPI4B1.2 (5V)
- net GND: now reaches RASPBERRYPI4B1.39 (GND)
Other:
- sheet HallSensor renamed HallSensor1
- added sheet HallSensor2 (hallsensor.kicad_sch)
- sheet HallSensor1 ports: added GND, SCL, SDA, VDD; removed none
- note added: "0.2.1"
- note added: "25.03.24"
- note added: "Luzian Raphael Aufdenblatten Tobias Muehlemann"
- note added: "Skógahöf Mainschematic"
- note added: "TODO"
- moved on the sheet: M1, M2, MotorHAT1, RASPBERRYPI4B1

Commit message: added Laserbarrier files and calculations
Parts:
- added M3: Lager ROT, symbol Motor:Motor_Servo
- added M4: Lager GRÜN, symbol Motor:Motor_Servo
- added M5: Lager BLAU, symbol Motor:Motor_Servo
- added M6: Zentrierschieber 1, symbol Motor:Motor_Servo
- added M7: Zentrierschieber 2, symbol Motor:Motor_Servo
- added ServoHAT1: ~, symbol Raspberry_4B:RaspberryPi4ServoHat
Connections:
- net +5V: now also ServoHAT1.1 (5V)
- net Displayshield/SCL: now also ServoHAT1.3 (SCL)
- net Displayshield/SDA: now also ServoHAT1.4 (SDA)
- net GND: now also ServoHAT1.2 (GND)
- net LaserSender/CTRL: now reaches RASPBERRYPI4B1.32 (GPIO_12_(PWM0))
- new net: M5.1 (PWM), ServoHAT1.8 (SIGNAL_2)
- new net: M3.2 (+), M4.2 (+), M5.2 (+), M6.2 (+), M7.2 (+), ServoHAT1.5 (VCC)
- new net: M3.3 (-), M4.3 (-), M5.3 (-), M6.3 (-), M7.3 (-), ServoHAT1.22 (GND)
- new net: M7.1 (PWM), ServoHAT1.10 (SIGNAL_4)
- new net: M3.1 (PWM), ServoHAT1.6 (SIGNAL_0)
- new net: M4.1 (PWM), ServoHAT1.7 (SIGNAL_1)
- new net: M6.1 (PWM), ServoHAT1.9 (SIGNAL_3)
Other:
- added sheet LaserSender (lasersend.kicad_sch)

Commit message: fixed main schematic :)
Other:
- added sheet LaserReceiver (laserreceiver.kicad_sch)
Changed lines of the file:
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@@
+    (stroke (width 0) (type default))
+  )
+  (wire (pts (xy 331.47 54.61) (xy 323.85 54.61))
     (stroke (width 0) (type default))
   )
@@
     (stroke (width 0) (type default))
   )
+  (wire (pts (xy 323.85 69.215) (xy 323.85 59.69))
+    (stroke (width 0) (type default))
+  )
   (wire (pts (xy 262.89 144.145) (xy 257.175 144.145))
     (stroke (width 0) (type default))
@@
     (stroke (width 0) (type default))
   )
+  (wire (pts (xy 323.85 59.69) (xy 331.47 59.69))
+    (stroke (width 0) (type default))
+  )
   (wire (pts (xy 181.61 85.09) (xy 191.77 85.09))
     (stroke (width 0) (type default))
@@
   )
   (wire (pts (xy 64.135 179.705) (xy 73.025 179.705))
+    (stroke (width 0) (type default))
+  )
+  (wire (pts (xy 323.85 54.61) (xy 323.85 46.99))
     (stroke (width 0) (type default))
   )
@@
     (fill (type none))
   )
+  (rectangle (start 314.325 53.975) (end 334.645 59.69)
+    (stroke (width 0) (type default) (color 255 0 0 1))
+    (fill (type none))
+  )
   (rectangle (start 233.68 161.925) (end 275.59 190.5)
     (stroke (width 0) (type default))
@@
   (text "Raspberry Display and Power\nIn-/Output" (at 234.315 166.37 0)
     (effects (font (size 1.27 1.27)) (justify left bottom))
+  )
+  (text "TODO" (at 325.12 58.42 0)
+    (effects (font (size 1.27 1.27) (color 255 0 0 1)) (justify left bottom))
   )
   (symbol (lib_id "Motor:Motor_Servo") (at 56.515 179.705 0) (mirror y) (unit 1)
@@
     )
   )
+  (symbol (lib_id "power:GND") (at 323.85 69.215 0) (unit 1)
+    (in_bom yes) (on_board yes) (dnp no) (fields_autoplaced)
+    (property "Reference" "#PWR058" (at 323.85 75.565 0)
+      (effects (font (size 1.27 1.27)) hide)
+    )
+    (property "Value" "GND" (at 323.85 73.66 0)
+      (effects (font (size 1.27 1.27)))
+    )
+    (property "Footprint" "" (at 323.85 69.215 0)
+      (effects (font (size 1.27 1.27)) hide)
+    )
+    (property "Datasheet" "" (at 323.85 69.215 0)
+      (effects (font (size 1.27 1.27)) hide)
+    )
+    (pin "1")
+    (instances
+      (project "mainschematic"
+        (path "/086318dd-19eb-4c26-88b2-e7f1a0e5d55a"
+          (reference "#PWR058") (unit 1)
+        )
+      )
+    )
+  )
   (symbol (lib_id "power:+5V") (at 287.02 47.625 0) (unit 1)
     (in_bom yes) (on_board yes) (dnp no) (fields_autoplaced)
@@
         (path "/086318dd-19eb-4c26-88b2-e7f1a0e5d55a"
           (reference "#PWR034") (unit 1)
+        )
+      )
+    )
+  )
+  (symbol (lib_id "power:+5V") (at 323.85 46.99 0) (unit 1)
+    (in_bom yes) (on_board yes) (dnp no) (fields_autoplaced)
+    (property "Reference" "#PWR057" (at 323.85 50.8 0)
+      (effects (font (size 1.27 1.27)) hide)
+    )
+    (property "Value" "+5V" (at 323.85 42.545 0)
+      (effects (font (size 1.27 1.27)))
+    )
+    (property "Footprint" "" (at 323.85 46.99 0)
+      (effects (font (size 1.27 1.27)) hide)
+    )
+    (property "Datasheet" "" (at 323.85 46.99 0)
+      (effects (font (size 1.27 1.27)) hide)
+    )
+    (pin "1")
+    (instances
+      (project "mainschematic"
+        (path "/086318dd-19eb-4c26-88b2-e7f1a0e5d55a"
+          (reference "#PWR057") (unit 1)
         )
       )
@@
       )
     )
+  )
+  (sheet (at 331.47 51.435) (size 12.7 12.065) (fields_autoplaced)
+    (stroke (width 0.1524) (type solid) (color 72 0 0 1))
+    (fill (color 255 255 194 1.0000))
+    (property "Sheetname" "LaserReceiver" (at 331.47 50.7234 0)
+      (effects (font (size 1.27 1.27)) (justify left bottom))
+    )
+    (property "Sheetfile" "laserreceiver.kicad_sch" (at 331.47 64.0846 0)
+      (effects (font (size 1.27 1.27)) (justify left top))
+    )
+    (pin "LGHT" input (at 331.47 57.15 180)
+      (effects (font (size 1.27 1.27)) (justify left))
+    )
+    (pin "VDD" input (at 331.47 54.61 180)
+      (effects (font (size 1.27 1.27)) (justify left))
+    )
+    (pin "GND" input (at 331.47 59.69 180)
+      (effects (font (size 1.27 1.27)) (justify left))
+    )
+    (instances
+      (project "mainschematic"
+        (path "/086318dd-19eb-4c26-88b2-e7f1a0e5d55a" (page "6"))
+      )
+    )
